File: Eagle/Schematics & Board Layout/Tx Board Schematic/T08-TxClicker.sch (EAGLE design)
At the start: 75 parts, among them U1 CC430F513X---RGZ48

Commit message: Tx-Schematic update
Parts:
- removed C30: DNI, rcl:C-EUC0603
- removed F1: PTC0603, SparkFun-PowerIC:PTC0603
- removed R10: 10k, QuadResistor:R603X42012
- removed R6: 0, rcl:R-US_R0603
- removed R7: DNI, rcl:R-US_R0603
- added L10: ~200nH, rcl-amber:LL0402
- added TP4, TP5, TP6, TP7, TP8: TEST-POINT3, SparkFun-Passives:TEST-POINT3
- JTAG: value (none) -> 6pin
- LED1: value (none) -> Blue
- LED2: value (none) -> Green
- LED3: value (none) -> Red
- LED4: value (none) -> Yellow
- Y1: value (none) -> 26MHz
Connections:
- removed net ADC: R6.1, R7.1, R9-1.2, R9-2.2, R9-3.2, R9-4.2
- removed net N$13: R10-1.2, R4.1, S4.1, U$5.P$1, U$5.P$3, U$5.P$4, U$5.P$5
- removed net N$17: R10-2.1, R10-3.2, S2.1, U$3.P$1, U$3.P$3, U$3.P$4, U$3.P$5
- removed net N$19: R10-1.1, R10-2.2, S3.1, U$4.P$1, U$4.P$3, U$4.P$4, U$4.P$5
- removed net P2.3: C30.1, R7.2, U$6G$5.P$1, U1.48
- net GND: now also R9-1.2, R9-2.2, R9-3.2, R9-4.2; no longer C30.2, R6.2
- net N$20: now also R4.1, S2.1, S3.1, S4.1, U$3.P$1, U$3.P$3, U$3.P$4, U$3.P$5, U$4.P$1, U$4.P$3, U$4.P$4, U$4.P$5, U$5.P$1, U$5.P$3, U$5.P$4, U$5.P$5; no longer R10-3.1
- net N$9: now also C15.1, C16.1, C17.1, C18.1, C19.1, C20.1, C21.1, L10.2, U1.27, U1.28, U1.31, U1.32, U1.34; no longer F1.1, U$2.V+
- net P1.7: now also TP7.1
- net P2.0: now also TP6.1
- net P2.1: now also TP5.1
- net P2.2: now also TP4.1
- net VCC: now also L10.1, TP8.1, U$2.V+; no longer C15.1, C16.1, C17.1, C18.1, C19.1, C20.1, C21.1, F1.2, U1.27, U1.28, U1.31, U1.32, U1.34
Other:
- note added: "50ohm Tline (if required)"
- note added: "Power Supply"
- note added: "ZD-1"
- note added: "ZD-2"
- note added: "ZD-3"
- note added: "ZD-4"
- note removed: "0ZCM0005FF2G"
- note removed: "50ohm Tline"
- moved on the sheet: C31, C32, C33, C34, C6, C7, C8, C9, JTAG, R1, R5, R9-1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

Commit message: Tx-Schematic Update
Changed pull-down to 10Meg, changed JTAG EMI cap from DNI to 2pF,
Annotated JTAG as Tag-Connect
Parts:
- removed U$6: ESDA6V1-5M6, TVS:ESDA6V1-5M6
- added D1: ESDA6V1-5M6, TVS:ESDA6V1-5M6
- C6, C7, C8: value 2pF/DNI -> 2pF
- R9: value 1MEG -> 10MEG
Connections:
- net GND: now also D1G$1.2; no longer U$6G$1.2
- net P1.7: now also D1G$4.P$1; no longer U$6G$1.1
- net P2.0: now also D1G$3.P$1; no longer U$6G$2.P$1
- net P2.1: now also D1G$2.P$1; no longer U$6G$3.P$1
- net P2.2: now also D1G$1.1; no longer U$6G$4.P$1
Other:
- note added: "Tag-Connect"
- note removed: "ZD-1"
- note removed: "ZD-2"
- note removed: "ZD-3"
- note removed: "ZD-4"
- moved on the sheet: C1, C10, C22
