File: Eagle/Schematics & Board Layout/Tx Board Schematic/T08-TxClicker.brd (EAGLE design)
At the start: 88.9 x 44.5 mm, 76 parts, among them U1 CC430F513X---RGZ48, Y1 26MHz

Commit message: Added GPIO TP
Parts:
- added TP10, TP11, TP12, TP13, TP14, TP15, TP16, TP17, TP18, TP9: TEST-POINT3, SparkFun-Passives:PAD.03X.03
Connections:
- new net N$12: TP9.P$1
- new net N$33: U1.43
- new net P1.0: TP12.P$1, U1.13
- new net P1.1: TP13.P$1, U1.12
- new net P1.2: TP14.P$1, U1.11
- new net P1.3: TP16.P$1, U1.10
- new net P1.4: TP15.P$1, U1.9
- new net P1.5: TP17.P$1, U1.6
- new net P1.6: TP18.P$1, U1.5
- new net P2.3: U1.48
- new net P2.4: U1.47
- new net P2.5: U1.46
- new net P2.6: TP10.P$1, U1.24
- new net P2.7: TP11.P$1, U1.23
- new net P3.0: U1.21
- new net P3.1: U1.20
- new net P3.6: U1.15
- new net P3.7: U1.14
Changed lines of the file:
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@@
 <?xml version="1.0" encoding="utf-8"?>
 <!DOCTYPE eagle SYSTEM "eagle.dtd">
-<eagle version="7.1.0">
+<eagle version="6.4">
 <drawing>
 <settings>
@@
 <pass name="Default">
 <param name="RoutingGrid" value="50mil"/>
-<param name="AutoGrid" value="1"/>
-<param name="Efforts" value="0"/>
-<param name="TopRouterVariant" value="1"/>
 <param name="tpViaShape" value="round"/>
 <param name="PrefDir.1" value="|"/>
@@
 <element name="TP8" library="SparkFun-Passives" package="PAD.03X.03" value="TEST-POINT3" x="-68.58" y="-43.18"/>
 <element name="D1" library="TVS" package="5X-TVS" value="ESDA6V1-5M6" x="-71.12" y="-43.18"/>
+<element name="TP9" library="SparkFun-Passives" package="PAD.03X.03" value="TEST-POINT3" x="-71.12" y="-45.72"/>
+<element name="TP10" library="SparkFun-Passives" package="PAD.03X.03" value="TEST-POINT3" x="-71.12" y="-48.26"/>
+<element name="TP11" library="SparkFun-Passives" package="PAD.03X.03" value="TEST-POINT3" x="-71.12" y="-50.8"/>
+<element name="TP12" library="SparkFun-Passives" package="PAD.03X.03" value="TEST-POINT3" x="-71.12" y="-53.34"/>
+<element name="TP13" library="SparkFun-Passives" package="PAD.03X.03" value="TEST-POINT3" x="-71.12" y="-55.88"/>
+<element name="TP14" library="SparkFun-Passives" package="PAD.03X.03" value="TEST-POINT3" x="-71.12" y="-58.42"/>
+<element name="TP15" library="SparkFun-Passives" package="PAD.03X.03" value="TEST-POINT3" x="-71.12" y="-60.96"/>
+<element name="TP16" library="SparkFun-Passives" package="PAD.03X.03" value="TEST-POINT3" x="-71.12" y="-63.5"/>
+<element name="TP17" library="SparkFun-Passives" package="PAD.03X.03" value="TEST-POINT3" x="-71.12" y="-66.04"/>
+<element name="TP18" library="SparkFun-Passives" package="PAD.03X.03" value="TEST-POINT3" x="-71.12" y="-68.58"/>
 </elements>
 <signals>
@@
 <wire x1="50.34" y1="30.508" x2="50.34" y2="31.008" width="0" layer="19" extent="1-1"/>
 </signal>
+<signal name="P1.6">
+<contactref element="U1" pad="5"/>
+<contactref element="TP18" pad="P$1"/>
+<wire x1="43.64" y1="33.008" x2="-71.12" y2="-68.58" width="0" layer="19" extent="1-1"/>
+</signal>
+<signal name="P1.5">
+<contactref element="U1" pad="6"/>
+<contactref element="TP17" pad="P$1"/>
+<wire x1="43.64" y1="32.508" x2="-71.12" y2="-66.04" width="0" layer="19" extent="1-1"/>
+</signal>
+<signal name="P1.4">
+<contactref element="U1" pad="9"/>
+<contactref element="TP15" pad="P$1"/>
+<wire x1="43.64" y1="31.008" x2="-71.12" y2="-60.96" width="0" layer="19" extent="1-1"/>
+</signal>
+<signal name="P1.3">
+<contactref element="U1" pad="10"/>
+<contactref element="TP16" pad="P$1"/>
+<wire x1="43.64" y1="30.508" x2="-71.12" y2="-63.5" width="0" layer="19" extent="1-1"/>
+</signal>
+<signal name="P1.2">
+<contactref element="U1" pad="11"/>
+<contactref element="TP14" pad="P$1"/>
+<wire x1="43.64" y1="30.008" x2="-71.12" y2="-58.42" width="0" layer="19" extent="1-1"/>
+</signal>
+<signal name="P1.1">
+<contactref element="U1" pad="12"/>
+<contactref element="TP13" pad="P$1"/>
+<wire x1="43.64" y1="29.508" x2="-71.12" y2="-55.88" width="0" layer="19" extent="1-1"/>
+</signal>
+<signal name="P1.0">
+<contactref element="U1" pad="13"/>
+<contactref element="TP12" pad="P$1"/>
+<wire x1="44.24" y1="28.908" x2="-71.12" y2="-53.34" width="0" layer="19" extent="1-1"/>
+</signal>
+<signal name="P3.7">
+<contactref element="U1" pad="14"/>
+</signal>
+<signal name="P3.6">
+<contactref element="U1" pad="15"/>
+</signal>
+<signal name="P3.1">
+<contactref element="U1" pad="20"/>
+</signal>
+<signal name="P3.0">
+<contactref element="U1" pad="21"/>
+</signal>
+<signal name="P2.7">
+<contactref element="U1" pad="23"/>
+<contactref element="TP11" pad="P$1"/>
+<wire x1="49.24" y1="28.908" x2="-71.12" y2="-50.8" width="0" layer="19" extent="1-1"/>
+</signal>
+<signal name="P2.6">
+<contactref element="U1" pad="24"/>
+<contactref element="TP10" pad="P$1"/>
+<wire x1="49.74" y1="28.908" x2="-71.12" y2="-48.26" width="0" layer="19" extent="1-1"/>
+</signal>
+<signal name="P2.3">
+<contactref element="U1" pad="48"/>
+</signal>
+<signal name="P2.4">
+<contactref element="U1" pad="47"/>
+</signal>
+<signal name="P2.5">
+<contactref element="U1" pad="46"/>
+</signal>
+<signal name="N$33">
+<contactref element="U1" pad="43"/>
+</signal>
+<signal name="N$12">
+<contactref element="TP9" pad="P$1"/>
+</signal>
 </signals>
