File: Eagle/Schematics & Board Layout/Tx Board Schematic/T08-TxClicker-Rev1a.sch (EAGLE design)
At the start: 83 parts, among them U1 CC430F513X---RGZ48, X1-DNI SMA-SMD, Y1 26MHz

Commit message: layout update
Parts:
- added R17: (no value), QuadResistor:R603X42012
Connections:
- new net N$19: R17-3.2, U1.2
- new net N$20: R17-4.2, U1.1
- new net N$7: R17-1.2, U1.4
- new net N$9: R17-2.2, U1.3
- net P1.7: now also R17-1.1; no longer U1.4
- net P2.0: now also R17-2.1; no longer U1.3
- net P2.1: now also R17-3.1; no longer U1.2
- net P2.2: now also R17-4.1; no longer U1.1
Other:
- moved on the sheet: TP4, TP5, TP6, TP7

Commit message: Button Example
Parts:
- S1, S2, S3, S4: value TOUCHPAD_SWITCH_COMBO -> SWITCH-MOMENTARY-212MM; device SparkFun-Electromechanical--edited:TOUCHPAD_SWITCH_COMBO -> SparkFun-Electromechanical--edited:SWITCH-MOMENTARY-212MM
Changed lines of the file:
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@@
 <part name="X1-DNI" library="con-coax" deviceset="SMA-SMD" device=""/>
 <part name="SUPPLY18" library="supply2" deviceset="GND" device=""/>
-<part name="S1" library="SparkFun-Electromechanical--edited" deviceset="TOUCHPAD_SWITCH_COMBO" device="" value="TOUCHPAD_SWITCH_COMBO"/>
-<part name="S2" library="SparkFun-Electromechanical--edited" deviceset="TOUCHPAD_SWITCH_COMBO" device="" value="TOUCHPAD_SWITCH_COMBO"/>
-<part name="S3" library="SparkFun-Electromechanical--edited" deviceset="TOUCHPAD_SWITCH_COMBO" device="" value="TOUCHPAD_SWITCH_COMBO"/>
-<part name="S4" library="SparkFun-Electromechanical--edited" deviceset="TOUCHPAD_SWITCH_COMBO" device="" value="TOUCHPAD_SWITCH_COMBO"/>
+<part name="S1" library="SparkFun-Electromechanical--edited" deviceset="SWITCH-MOMENTARY-2" device="12MM" value="SWITCH-MOMENTARY-212MM"/>
+<part name="S2" library="SparkFun-Electromechanical--edited" deviceset="SWITCH-MOMENTARY-2" device="12MM" value="SWITCH-MOMENTARY-212MM"/>
+<part name="S3" library="SparkFun-Electromechanical--edited" deviceset="SWITCH-MOMENTARY-2" device="12MM" value="SWITCH-MOMENTARY-212MM"/>
+<part name="S4" library="SparkFun-Electromechanical--edited" deviceset="SWITCH-MOMENTARY-2" device="12MM" value="SWITCH-MOMENTARY-212MM"/>
 <part name="R7" library="rcl-amber" deviceset="R" device="0603" value="0-DNI"/>
 <part name="U$1" library="tagConnect" deviceset="TC2030" device="-MCP"/>

Commit message: Arranging silkscreen
Parts:
- removed TP17: TEST-POINT3, SparkFun-Passives:TEST-POINT3
- added TP19, TP20, TP21, TP22, TP23, TP27, TP28: TEST-POINT3, SparkFun-Passives:TEST-POINT3
- LED1: value Blue -> (none)
- LED2: value Green -> (none)
- LED3: value Red -> (none)
- LED4: value Yellow -> (none)
- S1, S2, S3, S4: value SWITCH-MOMENTARY-212MM -> TOUCHPAD_SWITCH_COMBOSWITC_TOUCHPAD; device SparkFun-Electromechanical--edited:SWITCH-MOMENTARY-212MM -> button_TestFootprint:TOUCHPAD_SWITCH_COMBOSWITC_TOUCHPAD
Connections:
- removed net P1.0: TP9.1, U1.13
- removed net P1.1: TP10.1
- removed net P1.2: TP11.1
- removed net P1.3: TP12.1
- removed net P2.3: U1.48
- removed net P2.4: U1.47
- removed net P2.5: U1.46
- removed net P2.6: U1.24
- removed net P2.7: U1.23
- removed net P3.0: U1.21
- removed net P3.1: U1.20
- removed net P3.6: U1.15
- removed net P3.7: U1.14
- removed net P5.1: U1.43
- new net N$21: TP9.1, U1.17
- new net N$22: TP10.1, U1.13
- new net N$23: TP11.1, U1.14
- new net N$24: TP12.1, U1.15
- new net N$25: TP13.1, U1.16
- new net N$26: TP14.1, U1.18
- new net N$27: TP15.1, U1.19
- new net N$28: TP16.1, U1.20
- new net N$30: TP18.1, U1.23
- new net N$31: TP19.1, U1.24
- new net N$35: TP27.1, U1.47
- new net N$36: TP28.1, U1.48
- net N$11: now also S1.BASE@1, S1.BASE@2, S2.BASE@1, S2.BASE@2, S3.BASE@1, S3.BASE@2, S4.BASE@1, S4.BASE@2; no longer S1.1, S2.1, S3.1, S4.1
- net P1.4: no longer TP13.1
- net P1.7: now also S4.TOP@1, S4.TOP@2; no longer S4.2
- net P2.0: now also S3.TOP@1, S3.TOP@2; no longer S3.2
- net P2.1: now also S2.TOP@1, S2.TOP@2; no longer S2.2
- net P2.2: now also S1.TOP@1, S1.TOP@2; no longer S1.2
- net PJ.0/TDO: now also TP23.1
- net PJ.1/TDI/TCLK: now also TP22.1
- net PJ.2/TMS: now also TP21.1
- net PJ.3/TCK: now also TP20.1
Other:
- moved on the sheet: C13, C16, TP10, TP11, TP12, TP13, TP14, TP15, TP16, TP18, TP9

Commit message: And looking decent 0.o
Parts:
- removed R17: (no value), QuadResistor:R603X42012
- added D1: UCLAMP3304A, Semtech-TVS_Diode:UCLAMP3304A
- added R13, R14, R15, R16: 1k, rcl-amber:R0603
- added TP17, TP24, TP25, TP26: TEST-POINT3, SparkFun-Passives:TEST-POINT3
- LED1: value (none) -> Blue
- LED2: value (none) -> Green
- LED3: value (none) -> Yellow
- LED4: value (none) -> Red
Connections:
- removed net RST/SBWTDIO: C1.1, R12.1, U$1.RST/SBWTDIO
- net GND: now also D1G1.2, D1G2.2
- net N$10: now also LED2.C; no longer LED3.C
- net N$13: now also LED4.A; no longer LED1.A
- net N$14: now also LED3.A; no longer LED2.A
- net N$15: now also LED3.C; no longer LED2.C
- net N$16: now also LED2.A; no longer LED3.A
- net N$17: now also LED1.A; no longer LED4.A
- net N$18: now also LED4.C; no longer LED1.C
- net N$19: now also R14.2; no longer R17-3.2
- net N$20: now also R13.2; no longer R17-4.2
- net N$21: now also TP13.1; no longer TP9.1
- net N$22: now also TP9.1; no longer TP10.1
- net N$23: now also TP10.1; no longer TP11.1
- net N$24: now also TP11.1; no longer TP12.1
- net N$25: now also TP12.1; no longer TP13.1
- net N$7: now also R16.2; no longer R17-1.2
- net N$9: now also R15.2; no longer R17-2.2
- net P1.4: now also LED1.C; no longer LED4.C
- net P1.5/RX: now also TP26.1
- net P1.6/TX: now also TP17.1
- net P1.7: now also D1G3.P$1, R16.1; no longer R17-1.1
- net P2.0: now also D1G4.P$1, R15.1; no longer R17-2.1
- net P2.1: now also D1G1.1, R14.1; no longer R17-3.1
- net P2.2: now also D1G2.1, R13.1; no longer R17-4.1
- net RST/NMI/SBWTDIO: now also C1.1, R12.1, TP24.1, U$1.RST/SBWTDIO
- net TEST/SBWTCK: now also TP25.1
Other:
- moved on the sheet: LED1, LED2, LED3, LED4, TP10, TP11, TP12, TP13, TP9

Commit message: Move Tag Connect
Vectorized fonts, moved tag connect, added tp labels
Parts:
- TP1, TP10, TP11, TP12, TP13, TP14, TP15, TP16, TP17, TP18, TP19, TP2, TP20, TP21, TP22, TP23, TP24, TP25, TP26, TP27, TP28, TP3, TP5, TP6, TP7, TP8: value TEST-POINT3 -> (none)
- TP9: value TEST-POINT3 -> TP9
