File: Eagle/Schematics & Board Layout/Tx Board Schematic/T08-TxClicker-Rev1a.brd (EAGLE design)
At the start: 83.8 x 42.2 mm, 98 parts, among them U1 CC430F513X---RGZ48, X1-DNI SMA-SMD, Y1 26MHz

Commit message: Logo ftw?
Parts:
- moved TP1 5.70 mm to (53.6, 40.2)
