File: Eagle/Schematics & Board Layout/Tx Board Schematic/T08-TxClicker-Rev1a/T08-TxClicker-Rev1a.brd (EAGLE design)
At the start: 83.8 x 42.2 mm, 99 parts, among them U1 CC430F513X---RGZ48, X1-DNI SMA-SMD, Y1 26MHz

Commit message: ECE411 Presentation
Parts:
- removed C29: 16pF, rcl-amber:C0402
- removed L9: 5.6nH, rcl-amber:L0402
- added C100: 1.5pF, rcl-amber:C0402
- added R100: 0 Ohm, rcl-amber:R0402
- L10: value ~200nH -> 200nH
Connections:
- net ANTENNA: now also C100.P$2, R100.P$1; no longer C29.P$1, L9.P$2
- net GND: now also C100.P$1; no longer L9.P$1
- net N$12: now also R100.P$2; no longer C29.P$2
Changed lines of the file:
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@@
 <element name="TP3" library="SparkFun-Passives" package="PAD.03X.03" value="" x="59.69" y="1.905" smashed="yes" rot="R270"/>
 <element name="U$6" library="PCB_Antenna_915MHz-halseth" package="PCB_ANTENNA_915MHZ" value="PCB_ANTENNA_915MHZOSHP" x="62.7524" y="9.8806" smashed="yes" rot="R270"/>
-<element name="C29" library="rcl-amber" package="C0402" value="16pF" x="60.7314" y="9.8806" smashed="yes" rot="R180">
+<element name="R100" library="rcl-amber" package="R0402" value="0 Ohm" x="60.7314" y="9.8806" smashed="yes" rot="R180">
 <attribute name="NAME" x="61.0774" y="10.5204" size="0.254" layer="25" font="vector" rot="R180"/>
 <attribute name="VALUE" x="61.3314" y="10.4806" size="0.254" layer="27" rot="R180"/>
 </element>
-<element name="L9" library="rcl-amber" package="L0402" value="5.6nH" x="61.2394" y="8.6106" smashed="yes" rot="R90">
+<element name="C100" library="rcl-amber" package="C0402" value="1.5pF" x="61.2394" y="8.6106" smashed="yes" rot="R90">
 <attribute name="NAME" x="60.8632" y="8.0106" size="0.254" layer="25" font="vector" rot="R90"/>
 <attribute name="VALUE" x="61.8394" y="8.0106" size="0.254" layer="27" rot="R90"/>
@@
 <attribute name="NAME" x="12.5984" y="23.0124" size="0.508" layer="25" font="vector"/>
 </element>
-<element name="L10" library="rcl-amber" package="L0603" value="~200nH" x="51.0794" y="19.9136" smashed="yes" rot="R270">
+<element name="L10" library="rcl-amber" package="L0603" value="200nH" x="51.0794" y="19.9136" smashed="yes" rot="R270">
 <attribute name="NAME" x="51.7212" y="20.6958" size="0.508" layer="25" font="vector" rot="R270"/>
 <attribute name="VALUE" x="50.1194" y="20.8724" size="0.508" layer="27"/>
@@
 <contactref element="C10" pad="2"/>
 <contactref element="L8" pad="P$1"/>
-<contactref element="L9" pad="P$1"/>
+<contactref element="C100" pad="P$1"/>
 <contactref element="U$6" pad="GPLANE"/>
 <contactref element="C9" pad="2"/>
@@
 <signal name="ANTENNA">
 <contactref element="U$6" pad="ANT"/>
-<contactref element="C29" pad="P$1"/>
-<contactref element="L9" pad="P$2"/>
+<contactref element="R100" pad="P$1"/>
+<contactref element="C100" pad="P$2"/>
 <wire x1="61.2394" y1="9.1106" x2="61.2394" y2="9.8726" width="0.508" layer="1"/>
 <wire x1="61.2394" y1="9.8726" x2="61.2314" y2="9.8806" width="0.508" layer="1"/>
@@
 </signal>
 <signal name="N$12">
-<contactref element="C29" pad="P$2"/>
+<contactref element="R100" pad="P$2"/>
 <contactref element="L8" pad="P$2"/>
 <contactref element="C21" pad="P$1"/>
