File: Eagle/Schematics & Board Layout/Tx Board Schematic/T08-TxClicker-Rev1a/T08-TxClicker-Rev1a.sch (EAGLE design)
At the start: 99 parts, among them U1 CC430F513X---RGZ48, X1-DNI SMA-SMD, Y1 26MHz

Commit message: ECE411 Presentation
Parts:
- removed C29: 16pF, rcl-amber:C0402
- removed L9: 5.6nH, rcl-amber:LL0402
- added C100: 1.5pF, rcl-amber:C0402
- added R100: 0 Ohm, rcl-amber:R0402
- L10: value ~200nH -> 200nH
Connections:
- net ANTENNA: now also C100.2, R100.1; no longer C29.1, L9.2
- net GND: now also C100.1; no longer L9.1
- net N$12: now also R100.2; no longer C29.2
